Commit message: Update correct link inertias and weights

File: nexus_4wd_mecanum_description/urdf/nexus_4wd_mecanum.xacro (robot description, xacro)
@@ -23,11 +23,11 @@
     </collision>
     <inertial>
-      <!-- TODO Compute inertia based on cylinder -->
-      <origin xyz="0.0 0.0 0.0255" rpy="0 0 0"/>
-      <mass value="2.0"/>
-      <inertia
-        ixx="4.4744" ixy="0.03098" ixz="0.003647"
-        iyy="7.1624" iyz="0.1228"
-        izz="4.6155"/>
+      <!-- Inertia from CAD model, filled box assumption -->
+      <origin xyz="-0.01103 0 0.002" rpy="0 0 0"/>
+      <mass value="2.844"/>
+      <inertia
+        ixx="0.018819942" ixy="0" ixz="-0.000101519"
+        iyy="0.057333716" iyz="0"
+        izz="0.074201740"/>
     </inertial>
   </link>
@@ -52,11 +52,10 @@
     </collision>
     <inertial>
-      <origin xyz="0.0 0.0 0.0" rpy="0 0 0"/>
-      <mass value="0.0"/>
-      <!-- TODO Compute inertia based on cylinder -->
-      <inertia
-        ixx="4.4744" ixy="0.03098" ixz="0.003647"
-        iyy="7.1624" iyz="0.1228"
-        izz="4.6155"/>
+      <origin xyz="0 0.01221 0" rpy="0 0 0"/>
+      <mass value="0.055"/>
+      <inertia
+        ixx="0.000021370" ixy="0" ixz="0"
+        iyy="0.000009966" iyz="0"
+        izz="0.000021370"/>
     </inertial>
   </link>
@@ -81,11 +80,10 @@
     </collision>
     <inertial>
-      <origin xyz="0.0 0.0 0.0" rpy="0 0 0"/>
-      <mass value="0.0"/>
-      <!-- TODO Compute inertia based on cylinder -->
-      <inertia
-        ixx="4.4744" ixy="0.03098" ixz="0.003647"
-        iyy="7.1624" iyz="0.1228"
-        izz="4.6155"/>
+      <origin xyz="0 0.01221 0" rpy="0 0 0"/>
+      <mass value="0.055"/>
+      <inertia
+        ixx="0.000021370" ixy="0" ixz="0"
+        iyy="0.000009966" iyz="0"
+        izz="0.000021370"/>
     </inertial>
   </link>
@@ -110,11 +108,10 @@
     </collision>
     <inertial>
-      <origin xyz="0.0 0.0 0.0" rpy="0 0 0"/>
-      <mass value="0.0"/>
-      <!-- TODO Compute inertia based on cylinder -->
-      <inertia
-        ixx="4.4744" ixy="0.03098" ixz="0.003647"
-        iyy="7.1624" iyz="0.1228"
-        izz="4.6155"/>
+      <origin xyz="0 0.01221 0" rpy="0 0 0"/>
+      <mass value="0.055"/>
+      <inertia
+        ixx="0.000021370" ixy="0" ixz="0"
+        iyy="0.000009966" iyz="0"
+        izz="0.000021370"/>
     </inertial>
   </link>
@@ -139,11 +136,10 @@
     </collision>
     <inertial>
-      <origin xyz="0.0 0.0 0.0" rpy="0 0 0"/>
-      <mass value="0.0"/>
-      <!-- TODO Compute inertia based on cylinder -->
-      <inertia
-        ixx="4.4744" ixy="0.03098" ixz="0.003647"
-        iyy="7.1624" iyz="0.1228"
-        izz="4.6155"/>
+      <origin xyz="0 0.01221 0" rpy="0 0 0"/>
+      <mass value="0.055"/>
+      <inertia
+        ixx="0.000021370" ixy="0" ixz="0"
+        iyy="0.000009966" iyz="0"
+        izz="0.000021370"/>
     </inertial>
   </link>
@@ -170,9 +166,9 @@
       <origin xyz="0.0 0.0 0.0" rpy="0 0 0"/>
       <mass value="0.0"/>
-      <!-- TODO Compute inertia based on cylinder -->
-      <inertia
-        ixx="4.4744" ixy="0.03098" ixz="0.003647"
-        iyy="7.1624" iyz="0.1228"
-        izz="4.6155"/>
+      <!-- Inertia based on cylinder -->
+      <inertia
+        ixx="0.000324824" ixy="0" ixz="0"
+        iyy="0.000480000" iyz="0"
+        izz="0.000324824"/>
     </inertial>
   </link>
@@ -199,12 +195,11 @@
       <origin xyz="0.0 0.0 0.0" rpy="0 0 0"/>
       <mass value="0.0"/>
-      <!-- TODO Compute inertia based on cylinder -->
-      <inertia
-        ixx="4.4744" ixy="0.03098" ixz="0.003647"
-        iyy="7.1624" iyz="0.1228"
-        izz="4.6155"/>
-    </inertial>
-  </link>
-<!-- -->
+      <!-- Inertia based on cylinder -->
+      <inertia
+        ixx="0.000324824" ixy="0" ixz="0"
+        iyy="0.000480000" iyz="0"
+        izz="0.000324824"/>
+    </inertial>
+  </link>
   <joint name="upper_right_wheel_joint" type="fixed">
     <origin xyz="0 0.042 0" rpy="0 0 0" />
@@ -229,9 +224,9 @@
       <origin xyz="0.0 0.0 0.0" rpy="0 0 0"/>
       <mass value="0.0"/>
-      <!-- TODO Compute inertia based on cylinder -->
-      <inertia
-        ixx="4.4744" ixy="0.03098" ixz="0.003647"
-        iyy="7.1624" iyz="0.1228"
-        izz="4.6155"/>
+      <!-- Inertia based on cylinder -->
+      <inertia
+        ixx="0.000324824" ixy="0" ixz="0"
+        iyy="0.000480000" iyz="0"
+        izz="0.000324824"/>
     </inertial>
   </link>
@@ -258,9 +253,9 @@
       <origin xyz="0.0 0.0 0.0" rpy="0 0 0"/>
       <mass value="0.0"/>
-      <!-- TODO Compute inertia based on cylinder -->
-      <inertia
-        ixx="4.4744" ixy="0.03098" ixz="0.003647"
-        iyy="7.1624" iyz="0.1228"
-        izz="4.6155"/>
+      <!-- Inertia based on cylinder -->
+      <inertia
+        ixx="0.000324824" ixy="0" ixz="0"
+        iyy="0.000480000" iyz="0"
+        izz="0.000324824"/>
     </inertial>
   </link>

Commit message: Add gazebo plugin and parameter file to urdf
Minor correction to wheel links masses. Add the force based move plugin to command the robot from a
velocity command. Wheel joints are now continuous for the potential addition of the wheel rotation
visualization later on.

File: nexus_4wd_mecanum_description/urdf/nexus_4wd_mecanum.xacro (robot description, xacro)
@@ -8,4 +8,10 @@
   <material name="dark_grey"><color rgba="0.2 0.2 0.2 1.0" /></material>
   <material name="light_grey"><color rgba="0.4 0.4 0.4 1.0" /></material>
+  <link name="base_footprint"></link>
+  <joint name="base_link_joint" type="fixed">
+    <origin xyz="0 0 0.05" rpy="0 0 0" />
+    <parent link="base_footprint"/>
+    <child link="base_link" />
+  </joint>
   <link name="base_link">
     <visual>
@@ -144,8 +150,9 @@
     </inertial>
   </link>
-  <joint name="upper_left_wheel_joint" type="fixed">
+  <joint name="upper_left_wheel_joint" type="continuous">
     <origin xyz="0 0.042 0" rpy="0 0 0" />
     <parent link="upper_left_wheel_shaft"/>
     <child link="upper_left_wheel" />
+    <axis xyz="0 1 0"/>
   </joint>
   <link name="upper_left_wheel">
@@ -165,5 +172,5 @@
     <inertial>
       <origin xyz="0.0 0.0 0.0" rpy="0 0 0"/>
-      <mass value="0.0"/>
+      <mass value="0.3844"/>
       <!-- Inertia based on cylinder -->
       <inertia
@@ -173,8 +180,9 @@
     </inertial>
   </link>
-  <joint name="lower_left_wheel_joint" type="fixed">
+  <joint name="lower_left_wheel_joint" type="continuous">
     <origin xyz="0 0.042 0" rpy="0 0 0" />
     <parent link="lower_left_wheel_shaft"/>
     <child link="lower_left_wheel" />
+    <axis xyz="0 1 0"/>
   </joint>
   <link name="lower_left_wheel">
@@ -194,5 +202,5 @@
     <inertial>
       <origin xyz="0.0 0.0 0.0" rpy="0 0 0"/>
-      <mass value="0.0"/>
+      <mass value="0.3844"/>
       <!-- Inertia based on cylinder -->
       <inertia
@@ -202,8 +210,9 @@
     </inertial>
   </link>
-  <joint name="upper_right_wheel_joint" type="fixed">
+  <joint name="upper_right_wheel_joint" type="continuous">
     <origin xyz="0 0.042 0" rpy="0 0 0" />
     <parent link="upper_right_wheel_shaft"/>
     <child link="upper_right_wheel" />
+    <axis xyz="0 1 0"/>
   </joint>
   <link name="upper_right_wheel">
@@ -223,5 +232,5 @@
     <inertial>
       <origin xyz="0.0 0.0 0.0" rpy="0 0 0"/>
-      <mass value="0.0"/>
+      <mass value="0.3844"/>
       <!-- Inertia based on cylinder -->
       <inertia
@@ -231,8 +240,9 @@
     </inertial>
   </link>
-  <joint name="lower_right_wheel_joint" type="fixed">
+  <joint name="lower_right_wheel_joint" type="continuous">
     <origin xyz="0 0.042 0" rpy="0 0 0" />
     <parent link="lower_right_wheel_shaft"/>
     <child link="lower_right_wheel" />
+    <axis xyz="0 1 0"/>
   </joint>
   <link name="lower_right_wheel">
@@ -252,5 +262,5 @@
     <inertial>
       <origin xyz="0.0 0.0 0.0" rpy="0 0 0"/>
-      <mass value="0.0"/>
+      <mass value="0.3844"/>
       <!-- Inertia based on cylinder -->
       <inertia
@@ -316,3 +326,5 @@
     </visual>
   </link>
+  <!-- Include controller plugin for Gazebo -->
+  <xacro:include filename="$(find nexus_4wd_mecanum_description)/urdf/nexus_4wd_mecanum.gazebo" />
 </robot>
